File: Circuit - KiCad/PinguBot/PinguBot.kicad_sch (KiCad schematic)
At the start: 26 parts, among them J1 Jack-DC, J2 Conn_01x08_Pin, J3 Conn_01x08_Pin, U1 LM386, U3 LM7805_TO220, U4 TSOP45xx, U5 ESP32_DEVKITC

Commit message: Circuit Improvement
Parts:
- R3, R5: footprint Resistor_THT:R_Axial_DIN0204_L3.6mm_D1.6mm_P7.62mm_Horizontal -> Resistor_THT:R_Axial_DIN0207_L6.3mm_D2.5mm_P10.16mm_Horizontal
- U4: footprint OptoDevice:Vishay_MOLD-3Pin -> EESTN5:BORNERA3
Changed lines of the file:
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@@
 			)
 		)
-		(property "Footprint" "Resistor_THT:R_Axial_DIN0204_L3.6mm_D1.6mm_P7.62mm_Horizontal"
+		(property "Footprint" "Resistor_THT:R_Axial_DIN0207_L6.3mm_D2.5mm_P10.16mm_Horizontal"
 			(at 117.602 59.69 90)
 			(effects
@@
 			)
 		)
-		(property "Footprint" "OptoDevice:Vishay_MOLD-3Pin"
+		(property "Footprint" "EESTN5:BORNERA3"
 			(at 186.69 268.605 0)
 			(effects
@@
 			)
 		)
-		(property "Footprint" "Resistor_THT:R_Axial_DIN0204_L3.6mm_D1.6mm_P7.62mm_Horizontal"
+		(property "Footprint" "Resistor_THT:R_Axial_DIN0207_L6.3mm_D2.5mm_P10.16mm_Horizontal"
 			(at 219.71 255.778 90)
 			(effects
