File: Circuit - KiCad/PinguBot/PinguBot.kicad_sch (KiCad schematic)
At the start: 26 parts, among them J1 Jack-DC, J2 Conn_01x08_Pin, J3 Conn_01x08_Pin, U1 LM386, U3 LM7805_TO220, U4 TSOP45xx, U5 ESP32_DEVKITC

Commit message: Circuit Improvement | PCB Advanced
Parts:
- R4: footprint Resistor_THT:R_Axial_DIN0204_L3.6mm_D1.6mm_P7.62mm_Horizontal -> Resistor_THT:R_Axial_DIN0207_L6.3mm_D2.5mm_P7.62mm_Horizontal
Connections:
- net GND: now also Microphone1.1 (Pin_1), Speaker1.1 (Pin_1); no longer Microphone1.2 (Pin_2), Speaker1.2 (Pin_2)
- net Microphone ADC: now also Microphone1.2 (Pin_2); no longer Microphone1.1 (Pin_1)
- net SCL_DISPLAY: now also DisplayOled1.3 (Pin_3); no longer DisplayOled1.2 (Pin_2)
- net SDA_DISPLAY: now also DisplayOled1.2 (Pin_2); no longer DisplayOled1.3 (Pin_3)
- net at C1.2: now also Speaker1.2 (Pin_2); no longer Speaker1.1 (Pin_1)
Other:
- moved on the sheet: Speaker1
Changed lines of the file:
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@@
 	(wire
 		(pts
-			(xy 358.14 85.09) (xy 370.84 85.09)
+			(xy 358.14 85.09) (xy 381 85.09)
 		)
 		(stroke
@@
 	(wire
 		(pts
-			(xy 96.52 254) (xy 101.6 254)
+			(xy 381 68.58) (xy 381 58.42)
 		)
 		(stroke
@@
 	(wire
 		(pts
-			(xy 370.84 64.77) (xy 370.84 58.42)
-		)
-		(stroke
-			(width 0)
-			(type default)
-		)
-	)
-	(wire
-		(pts
 			(xy 119.38 50.8) (xy 119.38 55.88)
 		)
@@
 	(wire
 		(pts
-			(xy 96.52 256.54) (xy 101.6 256.54)
-		)
-		(stroke
-			(width 0)
-			(type default)
-		)
-	)
-	(wire
-		(pts
 			(xy 325.12 55.88) (xy 331.47 55.88)
 		)
@@
 	(wire
 		(pts
-			(xy 237.49 143.51) (xy 229.87 143.51)
+			(xy 381 85.09) (xy 381 71.12)
 		)
 		(stroke
@@
 	(wire
 		(pts
-			(xy 370.84 85.09) (xy 370.84 67.31)
+			(xy 237.49 143.51) (xy 229.87 143.51)
 		)
 		(stroke
@@
 	(wire
 		(pts
-			(xy 370.84 58.42) (xy 368.3 58.42)
+			(xy 97.79 256.54) (xy 101.6 256.54)
+		)
+		(stroke
+			(width 0)
+			(type default)
+		)
+	)
+	(wire
+		(pts
+			(xy 368.3 58.42) (xy 381 58.42)
+		)
+		(stroke
+			(width 0)
+			(type default)
+		)
+	)
+	(wire
+		(pts
+			(xy 97.79 254) (xy 101.6 254)
 		)
 		(stroke
@@
 	(global_label "SDA_DISPLAY"
 		(shape input)
-		(at 101.6 270.51 180)
+		(at 101.6 267.97 180)
 		(fields_autoplaced yes)
 		(effects
@@
 		)
 		(property "Intersheetrefs" "${INTERSHEET_REFS}"
-			(at 86.5195 270.51 0)
+			(at 86.5195 267.97 0)
 			(effects
 				(font
@@
 	(global_label "GND"
 		(shape input)
-		(at 96.52 256.54 180)
+		(at 97.79 254 180)
 		(fields_autoplaced yes)
 		(effects
@@
 		)
 		(property "Intersheetrefs" "${INTERSHEET_REFS}"
-			(at 89.6643 256.54 0)
+			(at 90.9343 254 0)
 			(effects
 				(font
@@
 	(global_label "SCL_DISPLAY"
 		(shape input)
-		(at 101.6 267.97 180)
+		(at 101.6 270.51 180)
 		(fields_autoplaced yes)
 		(effects
@@
 		)
 		(property "Intersheetrefs" "${INTERSHEET_REFS}"
-			(at 86.58 267.97 0)
+			(at 86.58 270.51 0)
 			(effects
 				(font
@@
 	(global_label "Microphone ADC"
 		(shape input)
-		(at 96.52 254 180)
+		(at 97.79 256.54 180)
 		(fields_autoplaced yes)
 		(effects
@@
 		)
 		(property "Intersheetrefs" "${INTERSHEET_REFS}"
-			(at 78.174 254 0)
+			(at 79.444 256.54 0)
 			(effects
 				(font
@@
 	(symbol
 		(lib_id "Connector:Screw_Terminal_01x02")
-		(at 375.92 64.77 0)
+		(at 375.92 71.12 180)
 		(unit 1)
 		(exclude_from_sim no)
@@
 		(dnp no)
 		(property "Reference" "Speaker1"
-			(at 379.222 64.77 0)
+			(at 372.618 71.12 0)
 			(effects
 				(font
@@
 		)
 		(property "Value" "Screw_Terminal_01x02"
-			(at 378.46 67.3099 0)
+			(at 373.38 68.5801 0)
 			(effects
 				(font
@@
 		)
 		(property "Footprint" "EESTN5:BORNERA2"
-			(at 375.92 64.77 0)
+			(at 375.92 71.12 0)
 			(effects
 				(font
@@
 		)
 		(property "Datasheet" "~"
-			(at 375.92 64.77 0)
+			(at 375.92 71.12 0)
 			(effects
 				(font
@@
 		)
 		(property "Description" "Generic screw terminal, single row, 01x02, script generated (kicad-library-utils/schlib/autogen/connector/)"
-			(at 375.92 64.77 0)
+			(at 375.92 71.12 0)
 			(effects
 				(font
@@
 			)
 		)
-		(property "Footprint" "Resistor_THT:R_Axial_DIN0204_L3.6mm_D1.6mm_P7.62mm_Horizontal"
+		(property "Footprint" "Resistor_THT:R_Axial_DIN0207_L6.3mm_D2.5mm_P7.62mm_Horizontal"
 			(at 340.868 73.66 90)
 			(effects

Commit message: Circuit Improvement
Parts:
- removed C1: 220μF, Capacitor_THT:CP_Axial_L10.0mm_D4.5mm_P15.00mm_Horizontal, symbol Device:C_Polarized
- removed C2: 10μF, Capacitor_THT:CP_Axial_L10.0mm_D4.5mm_P15.00mm_Horizontal, symbol Device:C_Polarized
- removed C3: 0.1yF, Capacitor_THT:CP_Axial_L10.0mm_D4.5mm_P15.00mm_Horizontal, symbol Device:C
- removed C4, C5: 1μf, Capacitor_THT:CP_Axial_L10.0mm_D4.5mm_P15.00mm_Horizontal, symbol Device:C
- removed C6: 0.1yF, Capacitor_THT:CP_Axial_L10.0mm_D4.5mm_P15.00mm_Horizontal, symbol Device:C_Polarized
- removed D2: LED, Capacitor_THT:C_Axial_L3.8mm_D2.6mm_P10.00mm_Horizontal, symbol Device:LED
- removed DisplayOled1: Screw_Terminal_01x04, Connector_PinSocket_2.54mm:PinSocket_1x04_P2.54mm_Vertical, symbol Connector:Screw_Terminal_01x04
- removed J1: Jack-DC, Connector_BarrelJack:BarrelJack_Kycon_KLDX-0202-xC_Horizontal, symbol Connector:Jack-DC
- removed J2, J3: Conn_01x08_Pin, Connector_PinHeader_2.54mm:PinHeader_1x08_P2.54mm_Vertical, symbol Connector:Conn_01x08_Pin
- removed Microphone1, MotorOne1, MotorTwo1, Speaker1: Screw_Terminal_01x02, EESTN5:BORNERA2, symbol Connector:Screw_Terminal_01x02
- removed R1: 10, Resistor_THT:R_Axial_DIN0207_L6.3mm_D2.5mm_P10.16mm_Horizontal, symbol Device:R
- removed R2: POT, EESTN5:BORNERA3, symbol EESTN5:POT
- removed R3: 100, Resistor_THT:R_Axial_DIN0207_L6.3mm_D2.5mm_P10.16mm_Horizontal, symbol Device:R
- removed R4: 1,2K, Resistor_THT:R_Axial_DIN0207_L6.3mm_D2.5mm_P7.62mm_Horizontal, symbol Device:R
- removed R5: 220, Resistor_THT:R_Axial_DIN0207_L6.3mm_D2.5mm_P10.16mm_Horizontal, symbol Device:R
- removed ServoMotorOne1, ServoMotorTwo1: Screw_Terminal_01x03, EESTN5:BORNERA3, symbol Connector:Screw_Terminal_01x03
- removed U1: LM386, Package_DIP:DIP-8_W7.62mm_Socket, symbol Amplifier_Audio:LM386
- removed U3: LM7805_TO220, Package_TO_SOT_THT:TO-220-3_Vertical, symbol Regulator_Linear:LM7805_TO220
- removed U4: TSOP45xx, EESTN5:BORNERA3, symbol Interface_Optical:TSOP45xx
- removed U5: ESP32_DEVKITC, EESTN5:ESP32_DEVKITC, symbol EESTN5:ESP32_DEVKITC
Connections:
- no-connect marks 27 -> 0
Other:
- added sheet Audio Amplifier (audio-amplifier.kicad_sch)
- added sheet Custom Microcontroller (custom-microcontroller.kicad_sch)
- added sheet External Devices (external-devices.kicad_sch)
- added sheet H Bridge (h-bridge.kicad_sch)
- added sheet Power Supply (power-supply.kicad_sch)
- note removed: "Audio Amplifier"
- note removed: "Dual H-Bridge and DC Motors"
- note removed: "IR Receiver"
- note removed: "Output Devices"
- note removed: "Power Supply | Jack Connector"
