File: Circuit - KiCad/PinguBot/_autosave-PinguBot.kicad_sch (KiCad schematic)
At the start: 26 parts, among them J1 Jack-DC, J2 Conn_01x08_Pin, J3 Conn_01x08_Pin, U1 LM386, U3 LM7805_TO220, U4 TSOP45xx, U5 ESP32_DEVKITC

Commit message: Circuit Improvement
Parts:
- R4: footprint Resistor_THT:R_Axial_DIN0204_L3.6mm_D1.6mm_P7.62mm_Horizontal -> Resistor_THT:R_Axial_DIN0207_L6.3mm_D2.5mm_P7.62mm_Horizontal
Changed lines of the file:
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@@
 			)
 		)
-		(property "Footprint" "Resistor_THT:R_Axial_DIN0204_L3.6mm_D1.6mm_P7.62mm_Horizontal"
+		(property "Footprint" "Resistor_THT:R_Axial_DIN0207_L6.3mm_D2.5mm_P7.62mm_Horizontal"
 			(at 340.868 73.66 90)
 			(effects
