File: Circuit - KiCad/PinguBot/PinguBot.kicad_pcb (KiCad board)
At the start: 2 copper layers, 150 x 150 mm, 26 parts, among them J1 Jack-DC, J2 Conn_01x08_Pin, J3 Conn_01x08_Pin, U1 LM386, U3 LM7805_TO220, U4 TSOP45xx, U5 ESP32_DEVKITC

Commit message: Circuit Improvement
Parts:
- R1, R4: footprint Resistor_THT:R_Axial_DIN0207_L6.3mm_D2.5mm_P10.16mm_Horizontal -> Resistor_THT:R_Axial_DIN0204_L3.6mm_D1.6mm_P7.62mm_Horizontal
- R3, R5: footprint Resistor_THT:R_Axial_DIN0204_L3.6mm_D1.6mm_P7.62mm_Horizontal -> Resistor_THT:R_Axial_DIN0207_L6.3mm_D2.5mm_P10.16mm_Horizontal
- U4: footprint OptoDevice:Vishay_MOLD-3Pin -> EESTN5:BORNERA3
- moved C6 666.9 mm to (99.7, 139.6), turned to 180 degrees
- moved R3 660.4 mm to (99.9, 131.4), turned to 0 degrees
- moved U4 629.6 mm to (124.7, 127.0), turned to 180 degrees
- moved ServoMotorOne1 561.2 mm to (32.8, 74.0), turned to 90 degrees
- moved ServoMotorTwo1 560.9 mm to (33.2, 91.2), turned to 90 degrees
- moved Microphone1 541.7 mm to (53.1, 106.4), turned to 0 degrees
- moved DisplayOled1 372.5 mm to (148.8, 73.8), turned to 180 degrees
- moved J3 360.9 mm to (106.4, 70.7), turned to 90 degrees
- moved J2 318.3 mm to (123.3, 45.6), turned to -90 degrees
- moved MotorTwo1 275.0 mm to (148.7, 52.9), turned to 90 degrees
- moved MotorOne1 273.7 mm to (148.6, 40.9), turned to 90 degrees
- moved D2 67.6 mm to (99.8, 148.2)
- moved R5 57.5 mm to (106.0, 147.9), turned to -90 degrees
- moved U5 44.7 mm to (127.7, 96.1), turned to 0 degrees
- moved C5 33.9 mm to (120.2, 147.9), turned to -90 degrees
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Routing:
- net 5V: track 78.5 -> 175.5 mm
- net Net-(U4-Vs): track 0.00 -> 31.9 mm
- net IR_DATA: track 0.00 -> 30.9 mm
- net Speaker DAC: track 81.4 -> 104.3 mm, vias 0 -> 1
- net VIN: track 40.7 -> 57.2 mm
- net Net-(D2-A): track 5.44 -> 6.25 mm
Other:
- board size 150 x 150 mm -> 136.8 x 150 mm

Commit message: Circuit Improvement
Parts:
- J2, J3: footprint Connector_PinSocket_2.54mm:PinSocket_1x08_P2.54mm_Vertical -> Connector_PinHeader_2.54mm:PinHeader_1x08_P2.54mm_Vertical
- R1: footprint Resistor_THT:R_Axial_DIN0204_L3.6mm_D1.6mm_P7.62mm_Horizontal -> Resistor_THT:R_Axial_DIN0207_L6.3mm_D2.5mm_P10.16mm_Horizontal
- R4: footprint Resistor_THT:R_Axial_DIN0204_L3.6mm_D1.6mm_P7.62mm_Horizontal -> Resistor_THT:R_Axial_DIN0207_L6.3mm_D2.5mm_P7.62mm_Horizontal
- moved DisplayOled1 70.2 mm to (83.8, 100.3), turned to 90 degrees
- moved C2 37.5 mm to (93.3, 129.8), turned to 180 degrees
- moved C1 28.8 mm to (72.4, 152.9)
- moved C3 28.8 mm to (86.3, 167.9)
- moved R1 28.8 mm to (79.6, 156.7)
- moved R2 28.8 mm to (59.5, 137.4)
- moved Speaker1 28.8 mm to (60.1, 152.2)
- moved ServoMotorOne1 24.7 mm to (57.4, 71.7)
- moved ServoMotorTwo1 24.7 mm to (57.8, 89.0)
- moved R4 24.3 mm to (93.3, 135.8), turned to 180 degrees
- moved MotorOne1 24.3 mm to (153.7, 64.7)
- moved MotorTwo1 22.8 mm to (153.6, 75.2)
- moved R3 21.7 mm to (115.2, 146.8)
- moved J1 19.9 mm to (159.2, 154.0), turned to 0 degrees
- moved U1 18.6 mm to (70.7, 139.8), turned to 0 degrees
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Routing:
- net 5V: track 175.5 -> 337.0 mm
- net 3.3V: track 0.00 -> 106.9 mm
- net S_Motor_OUT_2: track 0.00 -> 99.1 mm
- net S_Motor_OUT_1: track 0.00 -> 91.7 mm, vias 0 -> 1
- net Microphone ADC: track 0.00 -> 72.8 mm
- net MO4: track 0.00 -> 46.1 mm
- net SDA_DISPLAY: track 0.00 -> 43.6 mm
- net MO3: track 0.00 -> 38.0 mm
- net SCL_DISPLAY: track 0.00 -> 37.7 mm
- net MO2: track 0.00 -> 29.9 mm
- net MO1: track 0.00 -> 24.0 mm
- net Net-(R4-Pad2): track 37.1 -> 18.4 mm
- net Speaker DAC: track 104.3 -> 87.0 mm
- net STBY: track 0.00 -> 15.0 mm
- net MB2: track 0.00 -> 15.0 mm
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
Commit message: Circuit Improvement | PCB Advanced
Parts:
- moved MotorOne1 92.8 mm to (62.2, 49.4), turned to 180 degrees
- moved MotorTwo1 84.9 mm to (72.7, 49.4), turned to 180 degrees
- moved J2 78.7 mm to (52.4, 92.2), turned to 180 degrees
- moved Microphone1 68.6 mm to (121.2, 80.1)
- moved ServoMotorTwo1 67.1 mm to (121.3, 67.1)
- moved ServoMotorOne1 67.0 mm to (121.2, 51.4)
- moved J3 56.2 mm to (69.5, 92.2), turned to 180 degrees
- moved U5 48.8 mm to (96.4, 69.2), turned to 90 degrees
- moved J1 43.4 mm to (118.4, 139.2)
- moved C4 41.6 mm to (100.2, 127.9)
- moved C5 40.2 mm to (94.3, 127.9)
- moved U4 40.0 mm to (121.2, 93.5), turned to 90 degrees
- moved C6 37.8 mm to (103.5, 109.1), turned to 180 degrees
- moved R3 34.9 mm to (103.4, 113.9), turned to 180 degrees
- moved R5 34.8 mm to (83.1, 132.9)
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Connections:
- C1 pad 2: Net-(Speaker1-Pin_1) -> Net-(Speaker1-Pin_2)
- DisplayOled1 pad 2: SCL_DISPLAY -> SDA_DISPLAY
- DisplayOled1 pad 3: SDA_DISPLAY -> SCL_DISPLAY
- Microphone1 pad 1: Microphone ADC -> GND
- Microphone1 pad 2: GND -> Microphone ADC
- Speaker1 pad 1: Net-(Speaker1-Pin_1) -> GND
- Speaker1 pad 2: GND -> Net-(Speaker1-Pin_2)
Routing:
- net 3.3V: track 106.9 -> 23.7 mm
- net S_Motor_OUT_2: track 99.1 -> 18.2 mm
- net Speaker DAC: track 87.0 -> 165.5 mm, vias 1 -> 0
- net S_Motor_OUT_1: track 91.7 -> 16.1 mm, vias 1 -> 0
- net 5V: track 337.0 -> 263.8 mm
- net Microphone ADC: track 72.8 -> 13.4 mm
- net Net-(C2-Pad2): track 30.3 -> 5.88 mm
- net Net-(Speaker1-Pin_1): track 23.7 -> 0.00 mm
- net VIN: track 59.6 -> 37.8 mm
- net Net-(U4-Vs): track 32.6 -> 52.7 mm
- net Net-(Speaker1-Pin_2): track 0.00 -> 17.9 mm
- net SCL_DISPLAY: track 37.7 -> 23.9 mm
- net MO2: track 29.9 -> 43.5 mm
- net MO1: track 24.0 -> 37.3 mm
- net MO3: track 38.0 -> 50.3 mm
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Other:
- board size 136.8 x 150 mm -> 96.3 x 107.3 mm

Commit message: Circuit Improvement | Yay!
Parts:
- moved C2 7.20 mm to (87.6, 114.8)
- moved DisplayOled1 6.46 mm to (98.5, 110.5), turned to 0 degrees
- moved R4 5.41 mm to (84.9, 109.4)
- moved R3 4.22 mm to (103.0, 118.1), turned to 0 degrees
- moved J2 3.42 mm to (51.2, 95.4)
- moved J3 3.42 mm to (68.3, 95.5)
- moved Microphone1 3.42 mm to (120.0, 83.3)
- moved ServoMotorTwo1 3.42 mm to (120.1, 70.3)
- moved U5 3.42 mm to (95.2, 72.5)
- moved MotorOne1 3.42 mm to (61.0, 52.6)
- moved MotorTwo1 3.42 mm to (71.5, 52.6)
- moved ServoMotorOne1 3.42 mm to (120.0, 54.7)
- moved U4 3.42 mm to (120.0, 96.7)
- moved C6 3.16 mm to (103.1, 112.2), turned to 0 degrees
- moved C3 2.45 mm to (74.0, 143.1)
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Routing:
- net SCL_DISPLAY: track 23.9 -> 38.9 mm
- net SDA_DISPLAY: track 34.3 -> 44.4 mm
- net 5V: track 263.8 -> 254.4 mm
- net Net-(R4-Pad2): track 24.8 -> 21.2 mm
- net Speaker DAC: track 165.5 -> 163.1 mm
- net Net-(C3-Pad1): track 8.05 -> 5.63 mm
- net Net-(C2-Pad1): track 4.74 -> 6.55 mm
- net Net-(C2-Pad2): track 5.88 -> 4.21 mm
- net MA2: track 25.4 -> 24.8 mm
Other:
- board size 96.3 x 107.3 mm -> 96.3 x 104.8 mm
- board text added: "Invertir TSOP y poner una bornera a mi conveniencia Ponerle cooler al modelo 3d por si acaso"

Commit message: Circuit Improvement
Parts:
- moved C3 11.2 mm to (71.4, 132.2)
- moved D2 11.2 mm to (84.4, 122.1)
- moved R1 11.2 mm to (65.8, 122.0)
- moved Speaker1 11.2 mm to (47.6, 121.9)
- moved C1 11.2 mm to (59.2, 117.0)
- moved J2 11.2 mm to (48.6, 84.5)
- moved U1 11.2 mm to (58.1, 103.9)
- moved C2 11.2 mm to (85.0, 103.9)
- moved C4 11.2 mm to (97.6, 117.0)
- moved C5 11.2 mm to (91.7, 117.0)
- moved C6 11.2 mm to (100.4, 101.3)
- moved DisplayOled1 11.2 mm to (95.8, 99.6)
- moved J3 11.2 mm to (65.7, 84.6)
- moved Microphone1 11.2 mm to (117.4, 72.4)
- moved R2 11.2 mm to (47.6, 109.0)
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