File: Circuit - KiCad/Device/Device/Device.kicad_sch (KiCad schematic)
At the start: 14 parts, among them Q1 2N2219, U1 MCP73831-2-MC, U2 USB

Commit message: Circuit Improvement
Other:
- note added: "Second Circuit"
- note removed: "zweiter Stromkreis"
Changed lines of the file:
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@@
 		)
 	)
-	(text "zweiter Stromkreis\n"
+	(text "Second Circuit\n"
 		(exclude_from_sim no)
 		(at 103.124 40.386 0)
